Commit message: Add files via upload

File: dualarm_config/urdf/dualarm.urdf (robot description, URDF)
Before this commit: robot dualarm, 20 links, 19 joints
Links:
- removed link mani1_eef
- removed link mani2_link1
- added link mani1_eff, mass 0.26908; collision mesh filename=package://dualarm_config/meshes/mani1_eef.STL; visual mesh filename=package://dualarm_config/meshes/mani1_eef.STL
- added link mani2_link8, mass 0.10158; collision mesh filename=package://dualarm_config/meshes/mani2_link7.STL; visual mesh filename=package://dualarm_config/meshes/mani2_link7.STL
- link mani2_link2: mass 0.63538 -> 0.67076; geometry collision mesh filename=package://dualarm_config/meshes/mani2_link1.STL; visual mesh filename=package://dualarm_config/meshes/mani2_link1.STL
- link mani2_link3: mass 0.55009 -> 0.63538; geometry collision mesh filename=package://dualarm_config/meshes/mani2_link2.STL; visual mesh filename=package://dualarm_config/meshes/mani2_link2.STL
- link mani2_link4: mass 0.45928 -> 0.55009; geometry collision mesh filename=package://dualarm_config/meshes/mani2_link3.STL; visual mesh filename=package://dualarm_config/meshes/mani2_link3.STL
- link mani2_link5: mass 0.43981 -> 0.45928; geometry collision mesh filename=package://dualarm_config/meshes/mani2_link4.STL; visual mesh filename=package://dualarm_config/meshes/mani2_link4.STL
- link mani2_link6: mass 0.30699 -> 0.43981; geometry collision mesh filename=package://dualarm_config/meshes/mani2_link5.STL; visual mesh filename=package://dualarm_config/meshes/mani2_link5.STL
- link mani2_link7: mass 0.10158 -> 0.30699; geometry collision mesh filename=package://dualarm_config/meshes/mani2_link6.STL; visual mesh filename=package://dualarm_config/meshes/mani2_link6.STL
Joints:
- joint mani1_joint7: child mani1_eef -> mani1_eff; origin xyz=0 -0.167 0.0 rpy=1.5708 0 0 -> xyz=0 -0.175 0.0 rpy=1.5708 0 0
- joint mani2_fixed: child mani2_link1 -> mani2_link2
- joint mani2_joint1: child mani2_link2 -> mani2_link3; parent mani2_link1 -> mani2_link2
- joint mani2_joint2: child mani2_link3 -> mani2_link4; parent mani2_link2 -> mani2_link3
- joint mani2_joint3: child mani2_link4 -> mani2_link5; parent mani2_link3 -> mani2_link4
- joint mani2_joint4: child mani2_link5 -> mani2_link6; parent mani2_link4 -> mani2_link5
- joint mani2_joint5: child mani2_link6 -> mani2_link7; parent mani2_link5 -> mani2_link6
- joint mani2_joint6: child mani2_link7 -> mani2_link8; parent mani2_link6 -> mani2_link7
- joint mani2_joint7: parent mani2_link7 -> mani2_link8
